Commit message: commit

File: src/mppi_solver/mppi_solver/models/canadarm/urdf/floating_canadarm.urdf (robot description, URDF)
Before this commit: robot SSRMS_Canadarm2, 10 links, 9 joints
Links:
- link B1: geometry collision mesh filename=package://simulation/models/canadarm/meshes/joint_v3_0.stl scale=1.0 1.0 1.0; visual mesh filename=package://simulation/models/canadarm/meshes/joint_v3_0.dae scale=1.0 1.0 1.0
- link B2: geometry collision mesh filename=package://simulation/models/canadarm/meshes/joint_v3_0.stl scale=1.0 1.0 1.0; visual mesh filename=package://simulation/models/canadarm/meshes/joint_v3_0.dae scale=1.0 1.0 1.0
- link B3: geometry collision mesh filename=package://simulation/models/canadarm/meshes/joint_v3_0.stl scale=1.0 1.0 1.0; collision mesh filename=package://simulation/models/canadarm/meshes/joint_v3_0.stl scale=1.0 1.0 1.0
- link B4: geometry collision mesh filename=package://simulation/models/canadarm/meshes/joint_v3_0.stl scale=1.0 1.0 1.0; collision mesh filename=package://simulation/models/canadarm/meshes/link_joint_v2_1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 scale=1.0 1.0 1.0
- link B5: geometry collision mesh filename=package://simulation/models/canadarm/meshes/joint_v3_0.stl scale=1.0 1.0 1.0; visual mesh filename=package://simulation/models/canadarm/meshes/joint_v3_0.dae scale=1.0 1.0 1.0
- link B6: geometry collision mesh filename=package://simulation/models/canadarm/meshes/joint_v3_0.stl scale=1.0 1.0 1.0; visual mesh filename=package://simulation/models/canadarm/meshes/joint_v3_0.dae scale=1.0 1.0 1.0
- link Base_SSRMS: geometry collision mesh filename=package://simulation/models/canadarm/meshes/ee.stl scale=1.0 1.0 1.0; visual mesh filename=package://simulation/models/canadarm/meshes/ee.dae scale=1.0 1.0 1.0
- link EE_SSRMS: geometry collision mesh filename=package://simulation/models/canadarm/meshes/ee.stl scale=1.0 1.0 1.0; visual mesh filename=package://simulation/models/canadarm/meshes/ee.dae scale=1.0 1.0 1.0
- link ISS: geometry collision mesh filename=package://simulation/models/canadarm/meshes/iss.stl scale=1.0 1.0 1.0; visual mesh filename=package://simulation/models/canadarm/meshes/iss.dae scale=1.0 1.0 1.0

File: src/space_robots_gz/simulation/models/canadarm/urdf/floating_canadarm.urdf (robot description, URDF)
Before this commit: robot SSRMS_Canadarm2, 10 links, 9 joints
Links:
- link B1: geometry collision mesh filename=package://simulation/models/canadarm/meshes/joint_v3_0.stl scale=1.0 1.0 1.0; visual mesh filename=package://simulation/models/canadarm/meshes/joint_v3_0.dae scale=1.0 1.0 1.0
- link B2: geometry collision mesh filename=package://simulation/models/canadarm/meshes/joint_v3_0.stl scale=1.0 1.0 1.0; visual mesh filename=package://simulation/models/canadarm/meshes/joint_v3_0.dae scale=1.0 1.0 1.0
- link B3: geometry collision mesh filename=package://simulation/models/canadarm/meshes/joint_v3_0.stl scale=1.0 1.0 1.0; collision mesh filename=package://simulation/models/canadarm/meshes/joint_v3_0.stl scale=1.0 1.0 1.0
- link B4: geometry collision mesh filename=package://simulation/models/canadarm/meshes/joint_v3_0.stl scale=1.0 1.0 1.0; collision mesh filename=package://simulation/models/canadarm/meshes/link_joint_v2_1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 scale=1.0 1.0 1.0
- link B5: geometry collision mesh filename=package://simulation/models/canadarm/meshes/joint_v3_0.stl scale=1.0 1.0 1.0; visual mesh filename=package://simulation/models/canadarm/meshes/joint_v3_0.dae scale=1.0 1.0 1.0
- link B6: geometry collision mesh filename=package://simulation/models/canadarm/meshes/joint_v3_0.stl scale=1.0 1.0 1.0; visual mesh filename=package://simulation/models/canadarm/meshes/joint_v3_0.dae scale=1.0 1.0 1.0
- link Base_SSRMS: geometry collision mesh filename=package://simulation/models/canadarm/meshes/ee.stl scale=1.0 1.0 1.0; visual mesh filename=package://simulation/models/canadarm/meshes/ee.dae scale=1.0 1.0 1.0
- link EE_SSRMS: geometry collision mesh filename=package://simulation/models/canadarm/meshes/ee.stl scale=1.0 1.0 1.0; visual mesh filename=package://simulation/models/canadarm/meshes/ee.dae scale=1.0 1.0 1.0
- link ISS: geometry collision mesh filename=package://simulation/models/canadarm/meshes/iss.stl scale=1.0 1.0 1.0; visual mesh filename=package://simulation/models/canadarm/meshes/iss.dae scale=1.0 1.0 1.0

File: src/space_robots_gz/simulation/models/canadarm/urdf/floating_canadarm.urdf.xacro (robot description, xacro)
@@ -4,104 +4,15 @@
 The link CoM locations (with respect to link frame) are set to zero as the inertia tensor is defined with respect to the link frame in the paper.
  -->
-<robot name="floating canadarm" xmlns:xacro="http://wiki.ros.org/xacro">
+<robot name="SSRMS_Canadarm2" xmlns:xacro="http://wiki.ros.org/xacro">
   <!-- Gazebo - ROS2 Control macro -->
-  <xacro:include filename="$(find simulation)/models/canadarm/urdf/floating_canadarm_camera.gazebo.xacro" />
-  <xacro:floating_canadarm_gazebo command_interface="effort" />
+  <xacro:include filename="$(find simulation)/models/canadarm/urdf/floating_canadarm.gazebo.xacro" />
+  <xacro:floating_canadarm command_interface="effort" />
   <xacro:property name="PI" value="3.1415926535897931"/>
-  <link name="world" />
-  <joint name="world_to_vx" type="fixed">
-    <parent link="world"/>
-    <child link="v_x_link"/>
-    <origin xyz="0 0 0" rpy="0 0 0"/>
-  </joint>
-  <link name="v_x_link">
-    <inertial>
-      <mass value="0.00001"/>
-      <origin xyz="0 0 0" rpy="0 0 0"/>
-      <inertia ixx="1e-9" ixy="0" ixz="0" iyy="1e-9" iyz="0" izz="1e-9"/>
-    </inertial>
-  </link>
-  <joint name="v_x_joint" type="prismatic">
-    <parent link="v_x_link"/>
-    <child link="v_y_link"/>
-    <origin rpy="0 0 0" xyz="0 0 0"/>
-    <axis xyz="1 0 0"/>
-    <limit lower="-10000.0" upper="10000.0" effort="1000.0" velocity="5.0"/>
-  </joint>
-  <link name="v_y_link">
-    <inertial>
-      <mass value="0.00001"/>
-      <origin xyz="0 0 0" rpy="0 0 0"/>
-      <inertia ixx="1e-9" ixy="0" ixz="0" iyy="1e-9" iyz="0" izz="1e-9"/>
-    </inertial>
-  </link>
-  <joint name="v_y_joint" type="prismatic">
-    <parent link="v_y_link"/>
-    <child link="v_z_link"/>
-    <origin rpy="0 0 0" xyz="0 0 0"/>
-    <axis xyz="0 1 0"/>
-    <limit lower="-10000.0" upper="10000.0" effort="1000.0" velocity="5.0"/>
-  </joint>
-  <link name="v_z_link">
-    <inertial>
-      <mass value="0.00001"/>
-      <origin xyz="0 0 0" rpy="0 0 0"/>
-      <inertia ixx="1e-9" ixy="0" ixz="0" iyy="1e-9" iyz="0" izz="1e-9"/>
-    </inertial>
-  </link>
-  <joint name="v_z_joint" type="prismatic">
-    <parent link="v_z_link"/>
-    <child link="v_r_link"/>
-    <origin rpy="0 0 0" xyz="0.0 0 -0.0"/>
-    <axis xyz="0 0 1"/>
-    <limit lower="-10000.0" upper="10000.0" effort="1000.0" velocity="5.0"/>
-  </joint>
-  <link name="v_r_link">
-    <inertial>
-      <mass value="0.00001"/>
-      <origin xyz="0 0 0" rpy="0 0 0"/>
-      <inertia ixx="1e-9" ixy="0" ixz="0" iyy="1e-9" iyz="0" izz="1e-9"/>
-    </inertial>
-  </link>
-  <joint name="v_r_joint" type="revolute">
-    <parent link="v_r_link"/>
-    <child link="v_p_link"/>
-    <origin rpy="0 0 0" xyz="0.0 0 -0.0"/>
-    <axis xyz="1 0 0"/>
-    <limit lower="-6.28" upper="6.28" effort="1000.0" velocity="5.0"/>
-  </joint>
-  <link name="v_p_link">
-    <inertial>
-      <mass value="0.00001"/>
-      <origin xyz="0 0 0" rpy="0 0 0"/>
-      <inertia ixx="1e-9" ixy="0" ixz="0" iyy="1e-9" iyz="0" izz="1e-9"/>
-    </inertial>
-  </link>
-  <joint name="v_p_joint" type="revolute">
-    <parent link="v_p_link"/>
-    <child link="v_yaw_link"/>
-    <origin rpy="0 0 0" xyz="0.0 0 -0.0"/>
-    <axis xyz="0 1 0"/>
-    <limit lower="-6.28" upper="6.28" effort="1000.0" velocity="5.0"/>
-  </joint>
-    <link name="v_yaw_link">
-    <inertial>
-      <mass value="0.00001"/>
-      <origin xyz="0 0 0" rpy="0 0 0"/>
-      <inertia ixx="1e-9" ixy="0" ixz="0" iyy="1e-9" iyz="0" izz="1e-9"/>
-    </inertial>
-  </link>
-  <joint name="v_yaw_joint" type="revolute">
-    <parent link="v_yaw_link"/>
-    <child link="ISS"/>
-    <origin rpy="0 0 0" xyz="0.0 0 -0.0"/>
-    <axis xyz="0 0 1"/>
-    <limit lower="-6.28" upper="6.28" effort="1000.0" velocity="5.0"/>
-  </joint>
+  <!-- <link name="world"/> -->
   <link name="ISS">
     <inertial>
       <origin rpy="0 0 0" xyz="0 0 0"/>
-      <mass value="1000.0"/>
-      <inertia ixx="1" ixy="0" ixz="0" iyy="1" iyz="0" izz="1"/>
+      <mass value="100000.0"/>
+      <inertia ixx="69585.02" ixy="0" ixz="0" iyy="69585.02" iyz="0" izz="66666.664"/>
     </inertial>
     <visual>
@@ -391,5 +302,5 @@
       <origin rpy="0 -3.1415 0" xyz="0 0 0"/>
       <geometry>
-        <mesh filename="package://simulation/models/canadarm/meshes/ee.stl" scale="1.0 1.0 1.0" />
+        <mesh filename="package://simulation/models/canadarm/meshes/ee.stl" scale="1.0 1.0 0.95" />
       </geometry>
     </collision>
@@ -416,43 +327,5 @@
     <parent link="EE_SSRMS"/>
     <child link="EE_SSRMS_tip"/>
-    <origin rpy="0 ${PI} 0" xyz="0 0 -1.4"/>
-  </joint>
-  <joint name="head_camera_joint" type="fixed">
-    <parent link="EE_SSRMS_tip"/>
-    <child link="camera_link"/>
-    <origin rpy="0 ${-PI/2} 0" xyz="0.4 -0.004 -0.15"/>
-  </joint>
-  <link name="camera_link">
-    <inertial>
-      <origin xyz="0 0 0" rpy="0 0 0"/>
-      <mass value="0.001" />
-      <inertia ixx="9.1875e-09" ixy="0.0" ixz="0.0" iyy="9.1875e-09" iyz="0.0" izz="1.378125e-08"/>
-    </inertial>
-		<visual>
-      <origin rpy="0.0 0 0" xyz="0 0 0"/>
-      <geometry>
-        <box size="0.0005 0.0005 0.0005"/>
-      </geometry>
-      <material name="green"/>
-    </visual>
-	</link>
-  <joint name="base_camera_joint" type="fixed">
-    <parent link="B1"/>
-    <child link="base_camera_link"/>
-    <origin rpy="0 1.5707963267948966 0" xyz="-0.292 -0.003 -1.15"/>
-  </joint>
-  <link name="base_camera_link">
-    <inertial>
-      <origin rpy="0 0 0" xyz="0 0 0"/>
-      <mass value="0.001"/>
-      <inertia ixx="9.1875e-09" ixy="0.0" ixz="0.0" iyy="9.1875e-09" iyz="0.0" izz="1.378125e-08"/>
-    </inertial>
-    <visual>
-      <origin rpy="0.0 0 0" xyz="0 0 0"/>
-      <geometry>
-        <box size="0.0005 0.0005 0.0005"/>
-      </geometry>
-      <material name="green"/>
-    </visual>
-  </link>
+    <origin rpy="${PI} 0 0" xyz="0 0 -1.4"/>
+  </joint>
 </robot>
