Commit message: commit

File: src/space_robots_gz/simulation/models/ets_vii/urdf/ets_vii.urdf copy.xacro (robot description, xacro)
@@ -10,4 +10,9 @@
       </geometry>
     </visual>
+    <collision>
+      <geometry>
+         <box size="2 2 2" />
+      </geometry>
+    </collision>
     <inertial>
       <mass value="2552"/>
@@ -23,4 +28,9 @@
       <material name="white"/>
     </visual>
+    <collision>
+      <geometry>
+        <box size="0.65 0.65 0.03" />
+      </geometry>
+    </collision>
     <inertial>
       <mass value="0.01"/>
@@ -40,4 +50,9 @@
       </geometry>
     </visual>
+    <collision>
+      <geometry>
+        <box size="0.25 0.3 0.5" />
+      </geometry>
+    </collision>
     <inertial>
       <mass value="35"/>
